Commit message: rendered robot from the robot_description in Gazebo Harmonic using 2 launch files: for world and for robot

File: src/robot_description/urdf/robot.urdf (robot description, URDF)
Before this commit: robot arm_5dof, 10 links, 9 joints
Links:
- link base_link: mass None -> 2.0; geometry collision cylinder length=0.05 radius=0.08; visual cylinder length=0.05 radius=0.08
- link forearm_link: mass None -> 0.8; geometry collision cylinder length=0.25 radius=0.035; collision sphere radius=0.045
- link gripper_base_link: mass None -> 0.2; geometry collision box size=0.06 0.08 0.02; visual box size=0.06 0.08 0.02
- link gripper_left_finger: mass None -> 0.05; geometry collision box size=0.02 0.01 0.06; collision box size=0.02 0.015 0.03
- link gripper_right_finger: mass None -> 0.05; geometry collision box size=0.02 0.01 0.06; collision box size=0.02 0.015 0.03
- link shoulder_link: mass None -> 1.5; geometry collision cylinder length=0.08 radius=0.06; visual cylinder length=0.08 radius=0.06
- link tcp: mass None -> 0.001
- link upper_arm_link: mass None -> 1.2; geometry collision cylinder length=0.3 radius=0.04; collision sphere radius=0.05
- link wrist_1_link: mass None -> 0.4; geometry collision cylinder length=0.06 radius=0.035; visual cylinder length=0.06 radius=0.035
- link wrist_2_link: mass None -> 0.3; geometry collision cylinder length=0.04 radius=0.03; visual cylinder length=0.04 radius=0.03

Commit message: controlled model in Gazebo with Action sent from CLI to ros2_control follow_joint_trajectory

File: src/robot_description/urdf/robot.urdf (robot description, URDF)
Before this commit: robot arm_5dof, 10 links, 9 joints
Links:
- added link world
Joints:
- added joint world_joint: type fixed, parent world, child base_link, origin xyz=0 0 0 rpy=0 0 0
